File: SpeakerProtect/SpeakerProtect.kicad_pcb (KiCad board)
At the start: 2 copper layers, 39.4 x 74.3 mm, 44 parts, among them J1 POWER, J2 L OUT, J3 R OUT, J4 R IN, J5 L IN, K1 Relay_DPST-NO, Q1 TIP122*, Q2 BD140, Q3 BC549, Q4 BC559, Q5 BC549

Commit message: fixed issues
Parts:
- moved R13 5.03 mm to (114.6, 75.7), turned to 0 degrees
- moved R11 2.11 mm to (114.6, 73.5), turned to 0 degrees
Connections:
- Q2 pad 1: Net-(D1-K) -> Net-(JP1-B)
- Q2 pad 2: Net-(JP1-B) -> Net-(D1-K)
- Q4 pad 1: Net-(JP1-B) -> Net-(Q2-B)
- Q4 pad 3: Net-(Q2-B) -> Net-(JP1-B)
Routing:
- net Net-(Q2-B): track 19.4 -> 8.21 mm
- net Net-(D1-K): track 16.3 -> 25.6 mm
- net Net-(JP1-B): track 61.8 -> 66.2 mm
- net Net-(D12-A): track 53.7 -> 57.4 mm
- net Net-(Q5-C): track 11.6 -> 15.1 mm
- net /AC: track 11.7 -> 15.0 mm
- net /DC: track 28.7 -> 31.7 mm
- net Net-(D11-A): track 9.39 -> 11.7 mm
- net Net-(Q3-C): track 22.6 -> 20.3 mm
- net Net-(J3-P1-Pad1): track 19.0 -> 19.7 mm
Other:
- board text added: "Omit * and fit jumper if no Vreg needed"
- board text removed: "Omit * and fit jumper if no V reg needed"
