File: SpeakerProtect/SpeakerProtect.kicad_sch (KiCad schematic)
At the start: 43 parts, among them J1 POWER, J2 L OUT, J3 R OUT, J4 R IN, J5 L IN, K1 Relay_DPST-NO, Q1 TIP122*, Q2 BD140, Q3 BC549, Q4 BC559, Q5 BC549

Commit message: fixed issues
Connections:
- net at D1.1 (K), K1.A1, R14.2: now also Q2.2 (C); no longer Q2.1 (E)
- net at C4.1, JP1.2 (B), Q1.3 (E)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: now also Q2.1 (E), Q4.3 (E); no longer Q2.2 (C), Q4.1 (C)
- net at Q2.3 (B), R13.2: now also Q4.1 (C); no longer Q4.3 (E)
Changed lines of the file:
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@@
 		(lib_id "Transistor_BJT:BC559")
 		(at 144.78 71.12 0)
+		(mirror x)
 		(unit 1)
 		(exclude_from_sim no)
@@
 		(on_board yes)
 		(dnp no)
-		(fields_autoplaced yes)
 		(property "Reference" "Q4"
-			(at 149.86 69.8499 0)
+			(at 149.86 72.3901 0)
 			(effects
 				(font
@@
 		)
 		(property "Value" "BC559"
-			(at 149.86 72.3899 0)
+			(at 149.86 69.8501 0)
 			(effects
 				(font
@@
 		)
 		(property "Footprint" "Package_TO_SOT_THT:TO-92L_Inline_Wide"
-			(at 149.86 73.025 0)
+			(at 149.86 69.215 0)
 			(effects
 				(font
@@
 		(lib_id "Transistor_BJT:BD140")
 		(at 172.72 81.28 0)
+		(mirror x)
 		(unit 1)
 		(exclude_from_sim no)
@@
 		(on_board yes)
 		(dnp no)
-		(fields_autoplaced yes)
 		(property "Reference" "Q2"
-			(at 177.8 80.0099 0)
+			(at 177.8 82.5501 0)
 			(effects
 				(font
@@
 		)
 		(property "Value" "BD140"
-			(at 177.8 82.5499 0)
+			(at 177.8 80.0101 0)
 			(effects
 				(font
@@
 		)
 		(property "Footprint" "Package_TO_SOT_THT:TO-126-3_Vertical"
-			(at 177.8 83.185 0)
+			(at 177.8 79.375 0)
 			(effects
 				(font
